File: Video Board/VGABoard.brd (EAGLE design)
At the start: 12 parts, among them IC1 74LS541N

Commit message: trace changed
Routing:
- net GND: track 75.9 -> 80.2 mm
Changed lines of the file:
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@@
 <?xml version="1.0" encoding="utf-8"?>
 <!DOCTYPE eagle SYSTEM "eagle.dtd">
-<eagle version="6.4">
+<eagle version="9.2.0">
 <drawing>
 <settings>
 <setting alwaysvectorfont="no"/>
+<setting keepoldvectorfont="yes"/>
 <setting verticaltext="up"/>
 </settings>
@@
 <param name="dpMaxLengthDifference" value="10mm"/>
 <param name="dpGapFactor" value="2.5"/>
-<param name="checkGrid" value="0"/>
 <param name="checkAngle" value="0"/>
 <param name="checkFont" value="1"/>
 <param name="checkRestrict" value="1"/>
+<param name="checkStop" value="0"/>
+<param name="checkValues" value="0"/>
+<param name="checkNames" value="1"/>
+<param name="checkWireStubs" value="1"/>
+<param name="checkPolygonWidth" value="0"/>
 <param name="useDiameter" value="13"/>
 <param name="maxErrors" value="50"/>
@@
 <pass name="Default">
 <param name="RoutingGrid" value="50mil"/>
+<param name="AutoGrid" value="1"/>
+<param name="Efforts" value="0"/>
+<param name="TopRouterVariant" value="1"/>
 <param name="tpViaShape" value="round"/>
 <param name="PrefDir.1" value="|"/>
@@
 </autorouter>
 <elements>
-<element name="U$1" library="SparkFun-Connectors" package="DB15" value="DB15" x="19.05" y="40.64"/>
-<element name="C1" library="SparkFun-Capacitors" package="CAP-PTH-SMALLEZ" value="100nF" x="31.75" y="26.67" rot="R270"/>
-<element name="IC1" library="74xx-us" package="DIL20" value="74LS541N" x="20.32" y="15.875"/>
-<element name="R1" library="resistor" package="0204/5" value="1.5K" x="11.43" y="25.4" rot="R90"/>
-<element name="R2" library="resistor" package="0204/5" value="3K" x="13.97" y="25.4" rot="R90"/>
-<element name="R3" library="resistor" package="0204/5" value="1.5K" x="19.05" y="25.4" rot="R90"/>
-<element name="R4" library="resistor" package="0204/5" value="3K" x="21.59" y="25.4" rot="R90"/>
-<element name="R5" library="resistor" package="0204/5" value="1.5K" x="26.67" y="25.4" rot="R90"/>
-<element name="R6" library="resistor" package="0204/5" value="3K" x="29.21" y="25.4" rot="R90"/>
-<element name="R7" library="resistor" package="0204/5" value="180" x="8.89" y="25.4" rot="R270"/>
-<element name="R8" library="resistor" package="0204/5" value="180" x="16.51" y="25.4" rot="R270"/>
-<element name="R9" library="resistor" package="0204/5" value="180" x="24.13" y="25.4" rot="R270"/>
+<element name="U$1" library="SparkFun-Connectors" package="DB15" value="DB15" x="19.05" y="40.64">
+<attribute name="NAME" x="18.255" y="39.45" size="0.4064" layer="25" ratio="10"/>
+<attribute name="VALUE" x="18.36" y="40.245" size="0.4064" layer="27" ratio="10"/>
+</element>
+<element name="C1" library="SparkFun-Capacitors" package="CAP-PTH-SMALLEZ" value="100nF" x="31.75" y="26.67" rot="R270">
+<attribute name="NAME" x="33.655" y="27.94" size="0.6096" layer="25" rot="R270"/>
+<attribute name="VALUE" x="29.21" y="27.94" size="0.6096" layer="27" rot="R270"/>
+</element>
+<element name="IC1" library="74xx-us" package="DIL20" value="74LS541N" x="20.32" y="15.875">
+<attribute name="NAME" x="7.239" y="12.827" size="1.27" layer="25" rot="R90"/>
+<attribute name="VALUE" x="10.541" y="15.494" size="1.27" layer="27"/>
+</element>
+<element name="R1" library="resistor" package="0204/5" value="1.5K" x="11.43" y="25.4" rot="R90">
+<attribute name="NAME" x="10.2616" y="23.3934" size="0.9906" layer="25" ratio="10" rot="R90"/>
+<attribute name="VALUE" x="13.7414" y="23.2664" size="0.9906" layer="27" ratio="10" rot="R90"/>
+</element>
+<element name="R2" library="resistor" package="0204/5" value="3K" x="13.97" y="25.4" rot="R90">
+<attribute name="NAME" x="12.8016" y="23.3934" size="0.9906" layer="25" ratio="10" rot="R90"/>
+<attribute name="VALUE" x="16.2814" y="23.2664" size="0.9906" layer="27" ratio="10" rot="R90"/>
+</element>
+<element name="R3" library="resistor" package="0204/5" value="1.5K" x="19.05" y="25.4" rot="R90">
+<attribute name="NAME" x="17.8816" y="23.3934" size="0.9906" layer="25" ratio="10" rot="R90"/>
+<attribute name="VALUE" x="21.3614" y="23.2664" size="0.9906" layer="27" ratio="10" rot="R90"/>
+</element>
+<element name="R4" library="resistor" package="0204/5" value="3K" x="21.59" y="25.4" rot="R90">
+<attribute name="NAME" x="20.4216" y="23.3934" size="0.9906" layer="25" ratio="10" rot="R90"/>
+<attribute name="VALUE" x="23.9014" y="23.2664" size="0.9906" layer="27" ratio="10" rot="R90"/>
+</element>
+<element name="R5" library="resistor" package="0204/5" value="1.5K" x="26.67" y="25.4" rot="R90">
+<attribute name="NAME" x="25.5016" y="23.3934" size="0.9906" layer="25" ratio="10" rot="R90"/>
+<attribute name="VALUE" x="28.9814" y="23.2664" size="0.9906" layer="27" ratio="10" rot="R90"/>
+</element>
+<element name="R6" library="resistor" package="0204/5" value="3K" x="29.21" y="25.4" rot="R90">
+<attribute name="NAME" x="28.0416" y="23.3934" size="0.9906" layer="25" ratio="10" rot="R90"/>
+<attribute name="VALUE" x="31.5214" y="23.2664" size="0.9906" layer="27" ratio="10" rot="R90"/>
+</element>
+<element name="R7" library="resistor" package="0204/5" value="180" x="8.89" y="25.4" rot="R270">
+<attribute name="NAME" x="10.0584" y="27.4066" size="0.9906" layer="25" ratio="10" rot="R270"/>
+<attribute name="VALUE" x="6.5786" y="27.5336" size="0.9906" layer="27" ratio="10" rot="R270"/>
+</element>
+<element name="R8" library="resistor" package="0204/5" value="180" x="16.51" y="25.4" rot="R270">
+<attribute name="NAME" x="17.6784" y="27.4066" size="0.9906" layer="25" ratio="10" rot="R270"/>
+<attribute name="VALUE" x="14.1986" y="27.5336" size="0.9906" layer="27" ratio="10" rot="R270"/>
+</element>
+<element name="R9" library="resistor" package="0204/5" value="180" x="24.13" y="25.4" rot="R270">
+<attribute name="NAME" x="25.2984" y="27.4066" size="0.9906" layer="25" ratio="10" rot="R270"/>
+<attribute name="VALUE" x="21.8186" y="27.5336" size="0.9906" layer="27" ratio="10" rot="R270"/>
+</element>
 </elements>
 <signals>
@@
 <wire x1="11.43" y1="34.29" x2="11.43" y2="31.75" width="0.8128" layer="16"/>
 <wire x1="11.43" y1="31.75" x2="10.16" y2="30.48" width="0.8128" layer="16"/>
-<wire x1="10.16" y1="30.48" x2="7.62" y2="30.48" width="0.8128" layer="16"/>
-<wire x1="7.62" y1="30.48" x2="6.35" y2="29.21" width="0.8128" layer="16"/>
-<wire x1="6.35" y1="29.21" x2="6.35" y2="24.13" width="0.8128" layer="16"/>
-<wire x1="6.35" y1="24.13" x2="7.62" y2="22.86" width="0.8128" layer="16"/>
+<wire x1="10.16" y1="30.48" x2="3.81" y2="30.48" width="0.8128" layer="16"/>
+<wire x1="3.81" y1="30.48" x2="3.81" y2="26.67" width="0.8128" layer="16"/>
+<wire x1="3.81" y1="26.67" x2="7.62" y2="22.86" width="0.8128" layer="16"/>
 <wire x1="7.62" y1="22.86" x2="8.89" y2="22.86" width="0.8128" layer="16"/>
 <wire x1="18.17" y1="35.56" x2="20.46" y2="35.56" width="0" layer="19" extent="1-1"/>
@@
 </signal>
 </signals>
+<mfgpreviewcolors>
+<mfgpreviewcolor name="soldermaskcolor" color="0xC8008000"/>
+<mfgpreviewcolor name="silkscreencolor" color="0xFFFEFEFE"/>
+<mfgpreviewcolor name="backgroundcolor" color="0xFF282828"/>
+<mfgpreviewcolor name="coppercolor" color="0xFFFFBF00"/>
+<mfgpreviewcolor name="substratecolor" color="0xFF786E46"/>
+</mfgpreviewcolors>
 </board>
 </drawing>
